Commit message: fixed urdf with camera

File: urdf/gen3.urdf (robot description, URDF)
Before this commit: robot gen3, 19 links, 18 joints
Links:
- removed link base_link
- removed link world
- added link camera_color_frame
- added link camera_depth_frame
- added link camera_link
- added link gen3_link, mass 1.697; collision mesh filename=file:///opt/ros/humble/share/kortex_description/arms/gen3/7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; visual mesh filename=file:///opt/ros/humble/share/kortex_description/arms/gen3/7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
- link bracelet_link: mass 0.364 -> 0.5
Joints:
- removed joint base_joint
- added joint camera_module: type fixed, parent end_effector_link, child camera_link, origin xyz=0 0.05639 -0.00305 rpy=3.141592653589793 3.141592653589793 0
- added joint color_module: type fixed, parent end_effector_link, child camera_color_frame, origin xyz=0 0.05639 -0.00305 rpy=3.141592653589793 3.141592653589793 0
- added joint depth_module: type fixed, parent end_effector_link, child camera_depth_frame, origin xyz=0.0275 0.066 -0.00305 rpy=3.141592653589793 3.141592653589793 0
- added joint gen3_joint: type fixed, parent base_link, child gen3_link, origin xyz=-0.13186 0.0 0.320675 rpy=0 0 0
- joint joint_1: parent base_link -> gen3_link
